Commit message: updated description

File: photonfocus_camera_description/urdf/photonfocus_camera.xacro (robot description, xacro)
@@ -2,7 +2,6 @@
 <robot name="photonfocus_camera" xmlns:xacro="http://www.ros.org/wiki/xacro">
 <xacro:include filename="$(find photonfocus_camera_description)/urdf/materials.xacro" />
-<xacro:include filename="$(find photonfocus_camera_description)/urdf/photonfocus_camera.trans" />
 <xacro:include filename="$(find photonfocus_camera_description)/urdf/photonfocus_camera.gazebo" />
-<xacro:macro name="photonfocus_camera" params="parent camera_name">
+<xacro:macro name="photonfocus_camera" params="parent">
 	<link name="base_link">
 	  <inertial>
@@ -205,4 +204,6 @@
 	  <child link="Component5_1_1_1_1"/>
 	</joint>
+	<!-- extensions -->
+	<xacro:photonfocus_camera_gazebo/>
 </xacro:macro>
 </robot>

Commit message: updated typo

File: photonfocus_camera_description/urdf/photonfocus_camera.xacro (robot description, xacro)
@@ -1,5 +1,5 @@
 <?xml version="1.0" ?>
 <robot name="photonfocus_camera" xmlns:xacro="http://www.ros.org/wiki/xacro">
-    <xacro:macro name="storz_endoscope" params="endoscope_name robot_name parent">
+    <xacro:macro name="photonfocus_camera">
         <xacro:include filename="$(find photonfocus_camera_description)/urdf/materials.xacro" />
         <xacro:include filename="$(find photonfocus_camera_description)/urdf/photonfocus_camera.gazebo.xacro" />

Commit message: removed old spec

File: photonfocus_camera_description/urdf/photonfocus_camera.xacro (robot description, xacro)
@@ -5,7 +5,7 @@
         <xacro:include filename="$(find photonfocus_camera_description)/urdf/photonfocus_camera.gazebo.xacro" />
         <!--joint between {parent} and link_0-->
-        <joint name="${parent}_${endoscope_name}_joint" type="fixed">
+        <joint name="${parent}_photonfocus_joint" type="fixed">
             <parent link="${parent}"/>
-            <child link="${endoscope_name}_link_0"/>
+            <child link="link_0"/>
             <origin xyz="0 0 0" rpy="0 0 1.57079632679"/>
         </joint>
@@ -88,5 +88,5 @@
         <!-- TODO: add optical frame https://answers.ros.org/question/232534/gazebo-camera-frame-is-inconsistent-with-rviz-opencv-convention/ -->
         <!-- extensions -->
-        <xacro:storz_endoscope_gazebo endoscope_name="${endoscope_name}" robot_name="${robot_name}"/>
+        <xacro:storz_endoscope_gazebo/>
     </xacro:macro>
 </robot>

Commit message: updated moveit

File: photonfocus_camera_description/urdf/photonfocus_camera.xacro (robot description, xacro)
@@ -5,5 +5,5 @@
         <xacro:include filename="$(find photonfocus_camera_description)/urdf/photonfocus_camera.gazebo.xacro" />
         <!--joint between {parent} and link_0-->
-        <joint name="${parent}_photonfocus_joint" type="fixed">
+        <joint name="${parent}_photonfocus_camera_joint" type="fixed">
             <parent link="${parent}"/>
             <child link="link_0"/>
@@ -83,10 +83,10 @@
             <origin rpy="0 0 0" xyz="-0.003223 0.103999 0.00727"/>
             <parent link="link_2"/>
-            <child link="virtual_link_1"/>
+            <child link="link_cm"/>
         </joint>
         <link name="link_cm"/>
         <!-- TODO: add optical frame https://answers.ros.org/question/232534/gazebo-camera-frame-is-inconsistent-with-rviz-opencv-convention/ -->
         <!-- extensions -->
-        <xacro:storz_endoscope_gazebo/>
+        <xacro:photonfocus_camera_gazebo/>
     </xacro:macro>
 </robot>
