Commit message: added name prefix

File: med7pf/med7pf_description/urdf/med7pf.urdf.xacro (robot description, xacro)
@@ -11,4 +11,6 @@
     <xacro:arg name="origin_xyz" default="0 0 0"/>
     <xacro:arg name="origin_rpy" default="0 0 0"/>
+    <!-- Arguments for camera xacro -->
+    <xacro:arg name="camera_name" default="photonfocus_camera"/>
     <!-- fix to world -->
     <link name="world"/>
@@ -18,4 +20,4 @@
     </xacro:med7>
     <!-- insert photonfocus_camera -->
-    <xacro:photonfocus_camera parent="$(arg robot_name)_link_ee"/>
+    <xacro:photonfocus_camera parent="$(arg robot_name)_link_ee" robot_name="$(arg robot_name)" camera_name="$(arg camera_name)"/>
 </robot>

File: photonfocus_camera_description/urdf/photonfocus_camera.gazebo.xacro (robot description, xacro)
@@ -1,11 +1,8 @@
 <?xml version="1.0" ?>
 <robot name="photonfocus_camera" xmlns:xacro="http://www.ros.org/wiki/xacro" >
-<xacro:macro name="photonfocus_camera_gazebo">
-  <xacro:property name="body_color" value="Gazebo/Silver" />
-  <gazebo>
-    <plugin filename="libgazebo_ros_control.so" name="control"/>
-  </gazebo>
-  <gazebo reference="link_0">
-    <material>${body_color}</material>
+<xacro:macro name="photonfocus_camera_gazebo" params="camera_name robot_name">
+<!-- link 0 -->
+  <gazebo reference="${camera_name}_link_0">
+    <material>Gazebo/Grey</material>
     <mu1>0.2</mu1>
     <mu2>0.2</mu2>
@@ -13,16 +10,19 @@
     <gravity>true</gravity>
   </gazebo>
-  <gazebo reference="link_1">
-    <material>${body_color}</material>
+  <!-- link 1 -->
+  <gazebo reference="${camera_name}_link_1">
+    <material>Gazebo/Grey</material>
     <mu1>0.2</mu1>
     <mu2>0.2</mu2>
     <selfCollide>true</selfCollide>
   </gazebo>
-  <gazebo reference="link_2">
-    <material>${body_color}</material>
+  <!-- link 2 -->
+  <gazebo reference="${camera_name}_link_2">
+    <material>Gazebo/Grey</material>
     <mu1>0.2</mu1>
     <mu2>0.2</mu2>
     <selfCollide>true</selfCollide>
   </gazebo>
+  <!-- TODO: add camera -->
 </xacro:macro>
 </robot>

File: photonfocus_camera_description/urdf/photonfocus_camera.urdf.xacro (robot description, xacro)
@@ -4,7 +4,10 @@
     <!-- Include camera xacro -->
     <xacro:include filename="$(find photonfocus_camera_description)/urdf/photonfocus_camera.xacro"/>
+    <!--  Arguments for the med7 macro  -->
+    <xacro:arg name="camera_name" default="photonfocus_camera"/>
+    <xacro:arg name="robot_name" default="lbr"/>
     <!-- fix to world -->
     <link name="world"/>
     <!-- insert camera -->
-    <xacro:photonfocus_camera parent="world"/>
+    <xacro:photonfocus_camera camera_name="$(arg camera_name)" robot_name="$(arg robot_name)" parent="world"/>
 </robot>

File: photonfocus_camera_description/urdf/photonfocus_camera.xacro (robot description, xacro)
@@ -1,14 +1,15 @@
 <?xml version="1.0" ?>
 <robot name="photonfocus_camera" xmlns:xacro="http://www.ros.org/wiki/xacro">
-    <xacro:macro name="photonfocus_camera" params="parent">
+    <xacro:macro name="photonfocus_camera" params="camera_name robot_name parent">
+        <!-- include gazebo specifications -->
         <xacro:include filename="$(find photonfocus_camera_description)/urdf/materials.xacro" />
         <xacro:include filename="$(find photonfocus_camera_description)/urdf/photonfocus_camera.gazebo.xacro" />
         <!--joint between {parent} and link_0-->
-        <joint name="${parent}_photonfocus_camera_joint" type="fixed">
+        <joint name="${parent}_${camera_name}_joint" type="fixed">
             <parent link="${parent}"/>
-            <child link="link_0"/>
+            <child link="${camera_name}_link_0"/>
             <origin xyz="0 0 0" rpy="0 0 1.57079632679"/>
         </joint>
-        <link name="link_0">
+        <link name="${camera_name}_link_0">
             <inertial>
                 <origin rpy="0 0 0" xyz="0.0004526550759665437 0.0005013636920587692 0.01966691095028127"/>
@@ -30,10 +31,10 @@
             </collision>
         </link>
-        <joint name="joint_1" type="fixed">
+        <joint name="${camera_name}_joint_1" type="fixed">
             <origin rpy="0 0 0" xyz="-0.005763 0.000949 0.059647"/>
-            <parent link="link_0"/>
-            <child link="link_1"/>
+            <parent link="${camera_name}_link_0"/>
+            <child link="${camera_name}_link_1"/>
         </joint>
-        <link name="link_1">
+        <link name="${camera_name}_link_1">
             <inertial>
                 <origin rpy="0 0 0" xyz="-0.0029521431378939584 -0.015030724993614833 0.04528035169041975"/>
@@ -55,10 +56,10 @@
             </collision>
         </link>
-        <joint name="joint_2" type="fixed">
+        <joint name="${camera_name}_joint_2" type="fixed">
             <origin rpy="0 0 0" xyz="0.009 0.12 0.04"/>
-            <parent link="link_1"/>
-            <child link="link_2"/>
+            <parent link="${camera_name}_link_1"/>
+            <child link="${camera_name}_link_2"/>
         </joint>
-        <link name="link_2">
+        <link name="${camera_name}_link_2">
             <inertial>
                 <origin rpy="0 0 0" xyz="-0.003122152950603064 -0.036121615255736886 0.00045540214292298653"/>
@@ -80,13 +81,13 @@
             </collision>
         </link>
-        <joint name="joint_3" type="fixed">
+        <joint name="${camera_name}_joint_3" type="fixed">
             <origin rpy="0 0 0" xyz="-0.003223 0.103999 0.00727"/>
-            <parent link="link_2"/>
-            <child link="link_cm"/>
+            <parent link="${camera_name}_link_2"/>
+            <child link="${camera_name}_link_cm"/>
         </joint>
-        <link name="link_cm"/>
+        <link name="${camera_name}_link_cm"/>
         <!-- TODO: add optical frame https://answers.ros.org/question/232534/gazebo-camera-frame-is-inconsistent-with-rviz-opencv-convention/ -->
         <!-- extensions -->
-        <xacro:photonfocus_camera_gazebo/>
+        <xacro:photonfocus_camera_gazebo camera_name="${camera_name}" robot_name="${robot_name}"/>
     </xacro:macro>
 </robot>
